Commit message: safety_limits などを削除

File: universal_robot-kinetic-devel/ur_description/urdf/ur3.urdf.xacro (robot description, xacro)
@@ -21,8 +21,8 @@
     wrist_1_lower_limit:=${-pi}    wrist_1_upper_limit:=${pi}
     wrist_2_lower_limit:=${-pi}    wrist_2_upper_limit:=${pi}
-    wrist_3_lower_limit:=${-pi}    wrist_3_upper_limit:=${pi}
-    transmission_hw_interface:=hardware_interface/PositionJointInterface
+    wrist_3_lower_limit:=${-pi}    wrist_3_upper_limit:=${pi}">
+    <!-- transmission_hw_interface:=hardware_interface/PositionJointInterface
     safety_limits:=false safety_pos_margin:=0.15
-    safety_k_position:=20">
+    safety_k_position:=20" -->
     <!-- Inertia parameters -->
     <xacro:property name="base_mass" value="2.0" />  <!-- This mass might be incorrect -->
@@ -86,13 +86,7 @@
       <xacro:unless value="${joint_limited}">
         <limit lower="${-2.0 * pi}" upper="${2.0 * pi}" effort="330.0" velocity="2.16"/>
-        <xacro:if value="${safety_limits}">
-          <safety_controller soft_lower_limit="${-2.0 * pi + safety_pos_margin}" soft_upper_limit="${2.0 * pi - safety_pos_margin}" k_position="${safety_k_position}" k_velocity="0.0"/>
-        </xacro:if>
       </xacro:unless>
       <xacro:if value="${joint_limited}">
         <limit lower="${shoulder_pan_lower_limit}" upper="${shoulder_pan_upper_limit}" effort="330.0" velocity="2.16"/>
-        <xacro:if value="${safety_limits}">
-          <safety_controller soft_lower_limit="${shoulder_pan_lower_limit + safety_pos_margin}" soft_upper_limit="${shoulder_pan_upper_limit - safety_pos_margin}" k_position="${safety_k_position}" k_velocity="0.0"/>
-        </xacro:if>
       </xacro:if>
       <dynamics damping="0.0" friction="0.0"/>
@@ -123,13 +117,7 @@
       <xacro:unless value="${joint_limited}">
         <limit lower="${-2.0 * pi}" upper="${2.0 * pi}" effort="330.0" velocity="2.16"/>
-        <xacro:if value="${safety_limits}">
-          <safety_controller soft_lower_limit="${-2.0 * pi + safety_pos_margin}" soft_upper_limit="${2.0 * pi - safety_pos_margin}" k_position="${safety_k_position}" k_velocity="0.0"/>
-        </xacro:if>
       </xacro:unless>
       <xacro:if value="${joint_limited}">
         <limit lower="${shoulder_lift_lower_limit}" upper="${shoulder_lift_upper_limit}" effort="330.0" velocity="2.16"/>
-        <xacro:if value="${safety_limits}">
-          <safety_controller soft_lower_limit="${shoulder_lift_lower_limit + safety_pos_margin}" soft_upper_limit="${shoulder_lift_upper_limit - safety_pos_margin}" k_position="${safety_k_position}" k_velocity="0.0"/>
-        </xacro:if>
       </xacro:if>
       <dynamics damping="0.0" friction="0.0"/>
@@ -160,13 +148,7 @@
       <xacro:unless value="${joint_limited}">
         <limit lower="${-pi}" upper="${pi}" effort="150.0" velocity="3.15"/>
-        <xacro:if value="${safety_limits}">
-          <safety_controller soft_lower_limit="${-2.0 * pi + safety_pos_margin}" soft_upper_limit="${2.0 * pi - safety_pos_margin}" k_position="${safety_k_position}" k_velocity="0.0"/>
-        </xacro:if>
       </xacro:unless>
       <xacro:if value="${joint_limited}">
         <limit lower="${elbow_joint_lower_limit}" upper="${elbow_joint_upper_limit}" effort="150.0" velocity="3.15"/>
-        <xacro:if value="${safety_limits}">
-          <safety_controller soft_lower_limit="${elbow_joint_lower_limit + safety_pos_margin}" soft_upper_limit="${elbow_joint_upper_limit - safety_pos_margin}" k_position="${safety_k_position}" k_velocity="0.0"/>
-        </xacro:if>
       </xacro:if>
       <dynamics damping="0.0" friction="0.0"/>
@@ -197,13 +179,7 @@
       <xacro:unless value="${joint_limited}">
         <limit lower="${-2.0 * pi}" upper="${2.0 * pi}" effort="54.0" velocity="3.2"/>
-        <xacro:if value="${safety_limits}">
-          <safety_controller soft_lower_limit="${-2.0 * pi + safety_pos_margin}" soft_upper_limit="${2.0 * pi - safety_pos_margin}" k_position="${safety_k_position}" k_velocity="0.0"/>
-        </xacro:if>
       </xacro:unless>
       <xacro:if value="${joint_limited}">
         <limit lower="${wrist_1_lower_limit}" upper="${wrist_1_upper_limit}" effort="54.0" velocity="3.2"/>
-        <xacro:if value="${safety_limits}">
-          <safety_controller soft_lower_limit="${wrist_1_lower_limit + safety_pos_margin}" soft_upper_limit="${wrist_1_upper_limit - safety_pos_margin}" k_position="${safety_k_position}" k_velocity="0.0"/>
-        </xacro:if>
       </xacro:if>
       <dynamics damping="0.0" friction="0.0"/>
@@ -234,13 +210,7 @@
       <xacro:unless value="${joint_limited}">
         <limit lower="${-2.0 * pi}" upper="${2.0 * pi}" effort="54.0" velocity="3.2"/>
-        <xacro:if value="${safety_limits}">
-          <safety_controller soft_lower_limit="${-2.0 * pi + safety_pos_margin}" soft_upper_limit="${2.0 * pi - safety_pos_margin}" k_position="${safety_k_position}" k_velocity="0.0"/>
-        </xacro:if>
       </xacro:unless>
       <xacro:if value="${joint_limited}">
         <limit lower="${wrist_2_lower_limit}" upper="${wrist_2_upper_limit}" effort="54.0" velocity="3.2"/>
-        <xacro:if value="${safety_limits}">
-          <safety_controller soft_lower_limit="${wrist_2_lower_limit + safety_pos_margin}" soft_upper_limit="${wrist_2_upper_limit - safety_pos_margin}" k_position="${safety_k_position}" k_velocity="0.0"/>
-        </xacro:if>
       </xacro:if>
       <dynamics damping="0.0" friction="0.0"/>
@@ -270,14 +240,8 @@
       <axis xyz="0 1 0" />
       <xacro:unless value="${joint_limited}">
-        <limit lower="${-2.0 * pi}" upper="${2.0 * pi}" effort="54.0" velocity="3.2"/>
-        <xacro:if value="${safety_limits}">
-          <safety_controller soft_lower_limit="${-2.0 * pi + safety_pos_margin}" soft_upper_limit="${2.0 * pi - safety_pos_margin}" k_position="${safety_k_position}" k_velocity="0.0"/>
-        </xacro:if>
-      </xacro:unless>
+        <limit lower="${-2.0 * pi+1.23456}" upper="${2.0 * pi}" effort="54.0" velocity="3.2"/>
+        </xacro:unless>
       <xacro:if value="${joint_limited}">
         <limit lower="${wrist_3_lower_limit}" upper="${wrist_3_upper_limit}" effort="54.0" velocity="3.2"/>
-        <xacro:if value="${safety_limits}">
-          <safety_controller soft_lower_limit="${wrist_3_lower_limit + safety_pos_margin}" soft_upper_limit="${wrist_3_upper_limit - safety_pos_margin}" k_position="${safety_k_position}" k_velocity="0.0"/>
-        </xacro:if>
       </xacro:if>
       <dynamics damping="0.0" friction="0.0"/>
@@ -375,5 +339,5 @@
       <origin xyz="${0.016} ${0} ${0}" rpy="${0} ${0} ${0}" />
     </joint>
-    <xacro:ur_arm_transmission prefix="${prefix}" hw_interface="${transmission_hw_interface}" />
+    <!-- <xacro:ur_arm_transmission prefix="${prefix}" hw_interface="${transmission_hw_interface}" /> -->
     <xacro:ur_arm_gazebo prefix="${prefix}" />
     <!-- ROS base_link to UR 'Base' Coordinates transform -->

File: universal_robot-kinetic-devel/ur_description/urdf/ur3_robot.urdf.xacro (robot description, xacro)
@@ -17,5 +17,5 @@
     <parent link="world" />
     <child link = "base_link" />
-    <origin xyz="0.0 0.0 0.04" rpy="0.0 0.0 0.0" />
+    <origin xyz="0.0 0.0 0.0" rpy="0.0 0.0 0.0" />
   </joint>
 </robot>

Commit message: add zed_base_link

File: universal_robot-kinetic-devel/ur_description/urdf/ur3.urdf.xacro (robot description, xacro)
@@ -333,10 +333,19 @@
       </collision>
     </link>
+<!-- 14.48/2 -->
  <joint name="${prefix}zed_base_joint" type="fixed">
       <parent link="${prefix}camera_base" />
-      <child link = "${prefix}zbase_link" />
+      <child link = "${prefix}zed_base_link" />
       <!-- z= 0.008+0.01018-->
-      <origin xyz="${0.016} ${0} ${0}" rpy="${0} ${0} ${0}" />
-    </joint>
+      <origin xyz="${0.008+0.00724} ${0} ${0}" rpy="${0} ${0} ${0}" />
+    </joint>
+ <link name="${prefix}zed_base_link">
+      <collision>
+        <geometry>
+          <box size="0.01 0.01 0.01"/>
+        </geometry>
+        <origin rpy="0 0 0" xyz="0 0 0"/>
+      </collision>
+    </link>
     <!-- <xacro:ur_arm_transmission prefix="${prefix}" hw_interface="${transmission_hw_interface}" /> -->
     <xacro:ur_arm_gazebo prefix="${prefix}" />

Commit message: zed_base_link -> zbase_link

File: universal_robot-kinetic-devel/ur_description/urdf/ur3.urdf.xacro (robot description, xacro)
@@ -323,5 +323,5 @@
       <parent link="${prefix}camera_mount_link" />
       <child link = "${prefix}camera_base" />
-      <origin xyz="${0.065} ${0.0} ${0.000}" rpy="${pi} ${3*pi/2.0} ${0}" />
+      <origin xyz="${0.065} ${0.0} ${0.008+0.00724}" rpy="${pi} ${3*pi/2.0} ${0}" />
     </joint>
     <link name="${prefix}camera_base">
@@ -336,16 +336,8 @@
  <joint name="${prefix}zed_base_joint" type="fixed">
       <parent link="${prefix}camera_base" />
-      <child link = "${prefix}zed_base_link" />
+      <child link = "${prefix}zbase_link" />
       <!-- z= 0.008+0.01018-->
-      <origin xyz="${0.008+0.00724} ${0} ${0}" rpy="${0} ${0} ${0}" />
-    </joint>
- <link name="${prefix}zed_base_link">
-      <collision>
-        <geometry>
-          <box size="0.01 0.01 0.01"/>
-        </geometry>
-        <origin rpy="0 0 0" xyz="0 0 0"/>
-      </collision>
-    </link>
+      <origin xyz="${0} ${0} ${0}" rpy="${0} ${0} ${0}" />
+    </joint>
     <!-- <xacro:ur_arm_transmission prefix="${prefix}" hw_interface="${transmission_hw_interface}" /> -->
     <xacro:ur_arm_gazebo prefix="${prefix}" />

Commit message: dynpick の考慮

File: universal_robot-kinetic-devel/ur_description/urdf/ur3.urdf.xacro (robot description, xacro)
@@ -323,5 +323,5 @@
       <parent link="${prefix}camera_mount_link" />
       <child link = "${prefix}camera_base" />
-      <origin xyz="${0.065} ${0.0} ${0.008+0.00724}" rpy="${pi} ${3*pi/2.0} ${0}" />
+      <origin xyz="${0.065} ${0.0} ${0.008+0.008+0.00724+0.0325}" rpy="${pi} ${3*pi/2.0} ${0}" />
     </joint>
     <link name="${prefix}camera_base">
